File: Schematics/vibriskeeb.kicad_sch (KiCad schematic)
At the start: 123 parts, among them SW1 SW_Push, SW10 SW_Push, SW11 SW_Push, SW12 SW_Push, SW13 SW_Push, SW15 SW_Push, SW16 SW_Push, SW17 SW_Push, SW18 SW_Push, SW19 SW_Push, SW2 SW_Push, SW20 SW_Push, SW21 SW_Push, SW22 SW_Push, SW23 SW_Push, SW24 SW_Push, SW25 SW_Push, SW26 SW_Push, SW27 SW_Push, SW28 SW_Push, SW29 SW_Push, SW3 SW_Push, SW30 SW_Push, SW31 SW_Push, SW32 SW_Push, SW33 SW_Push, SW34 SW_Push, SW35 SW_Push, SW36 SW_Push, SW37 SW_Push, SW38 SW_Push, SW39 SW_Push, SW4 SW_Push, SW40 SW_Push, SW41 SW_Push, SW42 SW_Push, SW43 SW_Push, SW44 SW_Push, SW45 SW_Push, SW46 SW_Push, SW47 SW_Push, SW48 SW_Push, SW49 SW_Push, SW5 SW_Push, SW50 SW_Push, SW51 SW_Push, SW52 SW_Push, SW55 SW_Push, SW56 SW_Push, SW57 SW_Push, SW58 SW_Push, SW6 SW_Push, SW60 SW_Push, SW63 SW_Push, SW67 SW_Push, SW68 SW_Push, SW7 SW_Push, SW70 SW_Push, SW71 SW_Push, SW8 SW_Push, SW9 SW_Push, U1 RP2040-ZERO

Commit message: Add files via upload
Parts:
- removed D63, D67, D68, D70, D71: D, symbol Device:D
- removed SW63, SW67, SW68, SW70, SW71: SW_Push, symbol Switch:SW_Push
- added C1, C2, C3, C4: 100nF, symbol Device:C
- added D100, D101, D102, D103, D104, D105, D106, D107, D108, D109, D110, D111, D112, D113, D114, D115, D116, D117, D118, D119, D120, D121, D122, D123, D124, D125, D14, D63, D64, D65, D66, D67, D68, D69, D70, D71, D72, D73, D74, D75, D76, D77, D78, D79, D80, D81, D82, D83, D84, D85, D86, D87, D88, D89, D90, D91, D92, D93, D94, D95, D96, D97, D98, D99: LED, symbol Device:LED
- added D53, D54, D59, D61, D62: D, symbol Device:D
- added IC1, IC2, IC3, IC4: TLC5948APWPR, SOP65P640X120-25N, symbol TLC5948APWPR:TLC5948APWPR
- added R1, R2, R3, R4: 18K, symbol Device:R
- added SW14, SW53, SW54, SW59, SW61: SW_Push, symbol Switch:SW_Push
Connections:
- net C1: now also SW17.1, SW25.1, SW33.1, SW41.1, SW49.1, SW9.1, U1.9 (GP8); no longer SW15.1, SW29.1, U1.6 (GP5)
- net C2: now also SW10.1, SW18.1, SW26.1, SW34.1, SW42.1, SW50.1, U1.10 (GP9); no longer SW32.1, U1.7 (GP6)
- net C3: now also SW11.1, SW19.1, SW27.1, SW35.1, SW43.1, SW51.1, U1.11 (GP10), SW59.1; no longer SW17.1, SW33.1, SW34.1, U1.8 (GP7)
- net C4: now also SW12.1, SW20.1, SW28.1, SW44.1, SW52.1, U1.12 (GP11); no longer SW18.1, SW35.1, U1.9 (GP8)
- net C5: now also SW13.1, SW21.1, SW29.1, SW45.1, U1.13 (GP12), SW53.1, SW61.1; no longer SW19.1, SW38.1, U1.10 (GP9)
- net C6: now also SW22.1, SW30.1, SW38.1, SW46.1, U1.14 (GP13), SW14.1, SW54.1; no longer SW20.1, SW39.1, SW40.1, U1.11 (GP10)
- net C7: now also SW15.1, SW23.1, SW31.1, SW39.1, SW47.1, SW55.1, U1.15 (GP14); no longer SW21.1, SW41.1, SW42.1, U1.12 (GP11)
- net C8: now also SW16.1, SW24.1, SW32.1, SW40.1, SW48.1, SW56.1, U1.16 (GP15); no longer SW22.1, SW43.1, SW44.1, U1.13 (GP12)
- net R1: no longer D10.1 (K), D11.1 (K), D12.1 (K), D13.1 (K), D16.1 (K), D9.1 (K)
- net R2: now also D10.1 (K), D11.1 (K), D12.1 (K), D13.1 (K), D16.1 (K), D9.1 (K); no longer D18.1 (K), D19.1 (K), D20.1 (K), D21.1 (K), D22.1 (K), D23.1 (K), D24.1 (K), D25.1 (K), D26.1 (K), D27.1 (K), D28.1 (K), D30.1 (K)
- net R3: now also D18.1 (K), D19.1 (K), D20.1 (K), D21.1 (K), D22.1 (K), D23.1 (K), D24.1 (K), D25.1 (K); no longer D29.1 (K)
- net R4: now also D26.1 (K), D27.1 (K), D28.1 (K), D29.1 (K), D30.1 (K), D31.1 (K), D33.1 (K); no longer D34.1 (K), D36.1 (K), D38.1 (K), D40.1 (K), D42.1 (K), D44.1 (K), D46.1 (K), D48.1 (K), D50.1 (K), D52.1 (K), D56.1 (K)
- net R5: now also D34.1 (K), D35.1 (K), D36.1 (K), D37.1 (K), D38.1 (K), D39.1 (K), D40.1 (K), D41.1 (K); no longer D57.1 (K), D58.1 (K), D60.1 (K)
- net at D38.2 (A): now also SW37.2; no longer SW38.2
- net at SW18.2: now also D19.2 (A); no longer D18.2 (A)
- net at D49.2 (A): now also SW48.2; no longer SW49.2
- net at SW15.2: now also D16.2 (A); no longer D15.2 (A)
- net at SW46.2: now also D47.2 (A); no longer D46.2 (A)
- net at SW30.2: now also D31.2 (A); no longer D30.2 (A)
- net at SW39.2: now also D40.2 (A); no longer D39.2 (A)
- net at D44.2 (A): now also SW43.2; no longer SW44.2
- net at SW26.2: now also D27.2 (A); no longer D26.2 (A)
- net at SW28.2: now also D29.2 (A); no longer D28.2 (A)
- net at D25.2 (A): now also SW24.2; no longer SW25.2
- net at SW57.2: now also D58.2 (A); no longer D57.2 (A)
- net at D60.2 (A): now also SW59.2; no longer SW60.2
- net at SW19.2: now also D20.2 (A); no longer D19.2 (A)
- net at SW29.2: now also D30.2 (A); no longer D29.2 (A)
- net at D45.2 (A): now also SW44.2; no longer SW45.2
- net at SW17.2: now also D18.2 (A); no longer D17.2 (A)
- net at D23.2 (A): now also SW22.2; no longer SW23.2
- net at SW31.2: now also D32.2 (A); no longer D31.2 (A)
- net at SW58.2: now also D59.2 (A); no longer D58.2 (A)
- net at D22.2 (A): now also SW21.2; no longer SW22.2
- net at D52.2 (A): now also SW51.2; no longer SW52.2
- net at D37.2 (A): now also SW36.2; no longer SW37.2
- net at SW27.2: now also D28.2 (A); no longer D27.2 (A)
- net at D42.2 (A): now also SW41.2; no longer SW42.2
- net at SW40.2: now also D41.2 (A); no longer D40.2 (A)
- net at D21.2 (A): now also SW20.2; no longer SW21.2
- net at SW32.2: now also D33.2 (A); no longer D32.2 (A)
- net at D50.2 (A): now also SW49.2; no longer SW50.2
- net at SW33.2: now also D34.2 (A); no longer D33.2 (A)
- net at SW55.2: now also D56.2 (A); no longer D55.2 (A)
- net at D43.2 (A): now also SW42.2; no longer SW43.2
- net at D36.2 (A): now also SW35.2; no longer SW36.2
- net at D35.2 (A): now also SW34.2; no longer SW35.2
- net at SW47.2: now also D48.2 (A); no longer D47.2 (A)
- net at D51.2 (A): now also SW50.2; no longer SW51.2
- net at SW56.2: now also D57.2 (A); no longer D56.2 (A)
- net at D24.2 (A): now also SW23.2; no longer SW24.2
- net at SW16.2: now also D17.2 (A); no longer D16.2 (A)
- net +3.3V: now reaches U1.21 (3V3)
- net +3.3V: now also C1.2, C2.2, C3.2, C4.2, IC1.24 (VCC), IC2.24 (VCC), IC3.24 (VCC), IC4.24 (VCC)
- net GND: now reaches U1.22 (GND)
- net GND: now also C1.1, C2.1, C3.1, C4.1, IC1.1 (GND), IC1.25 (EP), IC2.1 (GND), IC2.25 (EP), IC3.1 (GND), IC3.25 (EP), IC4.1 (GND), IC4.25 (EP), R1.1, R2.1, R3.1, R4.1
- net +5V: now reaches U1.23 (5V)
- net +5V: now also D100.2 (A), D101.2 (A), D102.2 (A), D103.2 (A), D104.2 (A), D105.2 (A), D106.2 (A), D107.2 (A), D108.2 (A), D109.2 (A), D110.2 (A), D111.2 (A), D112.2 (A), D113.2 (A), D114.2 (A), D115.2 (A), D116.2 (A), D117.2 (A), D118.2 (A), D119.2 (A), D120.2 (A), D121.2 (A), D122.2 (A), D123.2 (A), D124.2 (A), D125.2 (A), D14.2 (A), D63.2 (A), D64.2 (A), D65.2 (A), D66.2 (A), D67.2 (A), D68.2 (A), D69.2 (A), D70.2 (A), D71.2 (A), D72.2 (A), D73.2 (A), D74.2 (A), D75.2 (A), D76.2 (A), D77.2 (A), D78.2 (A), D79.2 (A), D80.2 (A), D81.2 (A), D82.2 (A), D83.2 (A), D84.2 (A), D85.2 (A), D86.2 (A), D87.2 (A), D88.2 (A), D89.2 (A), D90.2 (A), D91.2 (A), D92.2 (A), D93.2 (A), D94.2 (A), D95.2 (A), D96.2 (A), D97.2 (A), D98.2 (A), D99.2 (A)
- removed net C10: SW10.1, SW24.1, SW47.1, SW48.1, U1.15 (GP14)
- removed net C11: SW11.1, SW25.1, SW49.1, SW50.1, U1.16 (GP15)
- removed net C12: SW12.1, SW26.1, SW51.1, SW52.1, U1.17 (GP26)
- removed net C13: SW13.1, SW27.1, SW31.1, U1.18 (GP27)
- removed net C14: SW28.1, SW55.1, SW56.1, U1.19 (GP28)
- removed net C15: SW16.1, SW30.1, U1.20 (GP29)
- removed net C9: SW23.1, SW45.1, SW46.1, SW9.1, U1.14 (GP13)
- new net: D53.2 (A), SW52.2
- new net: D62.2 (A), SW61.2
- new net: D61.2 (A), SW60.2
- new net: D54.2 (A), SW53.2
- new net: D26.2 (A), SW25.2
- new net: D15.2 (A), SW14.2
- new net: D39.2 (A), SW38.2
- new net: D46.2 (A), SW45.2
- new net: D55.2 (A), SW54.2
- new net DATA: IC1.2 (SIN), IC1.22 (SOUT), IC2.2 (SIN), IC2.22 (SOUT), IC3.2 (SIN), IC3.22 (SOUT), IC4.2 (SIN), IC4.22 (SOUT), U1.17 (GP26)
- new net GSCLK: IC1.21 (GSCLK), IC2.21 (GSCLK), IC3.21 (GSCLK), IC4.21 (GSCLK), U1.20 (GP29)
- new net IREF: IC1.23 (IREF), IC2.23 (IREF), IC3.23 (IREF), IC4.23 (IREF), R1.2, R2.2, R3.2, R4.2
- new net LAT: IC1.4 (LAT), IC2.4 (LAT), IC3.4 (LAT), IC4.4 (LAT), U1.19 (GP28)
- new net OUT0: D110.1 (K), D14.1 (K), D78.1 (K), D94.1 (K), IC1.5 (OUT0), IC2.5 (OUT0), IC3.5 (OUT0), IC4.5 (OUT0)
- new net OUT1: D112.1 (K), D63.1 (K), D80.1 (K), D96.1 (K), IC1.6 (OUT1), IC2.6 (OUT1), IC3.6 (OUT1), IC4.6 (OUT1)
- new net OUT10: D115.1 (K), D72.1 (K), D83.1 (K), D99.1 (K), IC1.15 (OUT10), IC2.15 (OUT10), IC3.15 (OUT10), IC4.15 (OUT10)
- new net OUT11: D101.1 (K), D117.1 (K), D73.1 (K), D85.1 (K), IC1.16 (OUT11), IC2.16 (OUT11), IC3.16 (OUT11), IC4.16 (OUT11)
- new net OUT12: D103.1 (K), D119.1 (K), D74.1 (K), D87.1 (K), IC1.17 (OUT12), IC2.17 (OUT12), IC3.17 (OUT12), IC4.17 (OUT12)
- new net OUT13: D105.1 (K), D121.1 (K), D75.1 (K), D89.1 (K), IC1.18 (OUT13), IC2.18 (OUT13), IC3.18 (OUT13), IC4.18 (OUT13)
- new net OUT14: D107.1 (K), D123.1 (K), D76.1 (K), D91.1 (K), IC1.19 (OUT14), IC2.19 (OUT14), IC3.19 (OUT14), IC4.19 (OUT14)
- new net OUT15: D109.1 (K), D125.1 (K), D77.1 (K), D93.1 (K), IC1.20 (OUT15), IC2.20 (OUT15), IC3.20 (OUT15), IC4.20 (OUT15)
- new net OUT2: D114.1 (K), D64.1 (K), D82.1 (K), D98.1 (K), IC1.7 (OUT2), IC2.7 (OUT2), IC3.7 (OUT2), IC4.7 (OUT2)
- new net OUT3: D100.1 (K), D116.1 (K), D65.1 (K), D84.1 (K), IC1.8 (OUT3), IC2.8 (OUT3), IC3.8 (OUT3), IC4.8 (OUT3)
- new net OUT4: D102.1 (K), D118.1 (K), D66.1 (K), D86.1 (K), IC1.9 (OUT4), IC2.9 (OUT4), IC3.9 (OUT4), IC4.9 (OUT4)
- new net OUT5: D104.1 (K), D120.1 (K), D67.1 (K), D88.1 (K), IC1.10 (OUT5), IC2.10 (OUT5), IC3.10 (OUT5), IC4.10 (OUT5)
- new net OUT6: D106.1 (K), D122.1 (K), D68.1 (K), D90.1 (K), IC1.11 (OUT6), IC2.11 (OUT6), IC3.11 (OUT6), IC4.11 (OUT6)
- new net OUT7: D108.1 (K), D124.1 (K), D69.1 (K), D92.1 (K), IC1.12 (OUT7), IC2.12 (OUT7), IC3.12 (OUT7), IC4.12 (OUT7)
- new net OUT8: D111.1 (K), D70.1 (K), D79.1 (K), D95.1 (K), IC1.13 (OUT8), IC2.13 (OUT8), IC3.13 (OUT8), IC4.13 (OUT8)
- new net OUT9: D113.1 (K), D71.1 (K), D81.1 (K), D97.1 (K), IC1.14 (OUT9), IC2.14 (OUT9), IC3.14 (OUT9), IC4.14 (OUT9)
- new net R6: D42.1 (K), D43.1 (K), D44.1 (K), D45.1 (K), D46.1 (K), D47.1 (K), D48.1 (K), D49.1 (K), U1.6 (GP5)
- new net R7: D50.1 (K), D51.1 (K), D52.1 (K), D53.1 (K), D54.1 (K), D55.1 (K), D56.1 (K), D57.1 (K), U1.7 (GP6)
- new net R8: D58.1 (K), D59.1 (K), D60.1 (K), D61.1 (K), D62.1 (K), U1.8 (GP7)
- new net SCLK: IC1.3 (SCLK), IC2.3 (SCLK), IC3.3 (SCLK), IC4.3 (SCLK), U1.18 (GP27)
Other:
- moved on the sheet: U1
